File: pcbs/40%.kicad_pcb (KiCad board)
At the start: 2 copper layers, 246.7 x 79.8 mm, 102 parts

Commit message: merge commit 1
Parts:
- removed the G*** at (210.5, 146.5)
- removed the G*** at (138.5, 149.0)
- removed the G*** at (287.5, 151.0)
- added G***: LOGO, LOGO, F.Cu at (213.0, 148.0)
- added G***: LOGO, LOGO, B.Cu at (216.1, 147.6)
- S1, S10, S11, S12, S13, S14, S15, S16, S17, S18, S19, S2, S20, S21, S22, S23, S24, S25, S26, S27, S28, S29, S3, S30, S31, S32, S33, S34, S35, S36, S37, S38, S39, S4, S40, S41, S42, S43, S44, S45, S5, S6, S7, S8, S9: footprint ceoloide:switch_mx -> smd2:switch_mx_sans-silk
Other:
- board text added: "4ourty - by theb0b 7/19/26"
- board text added: "Face Down"
- board text added: "JST"
- board text added: "MCU"
- board text added: "Power"
- board text added: "Reset"
